File: PCBs_schematics/Rover.sch (KiCad schematic (older format))
At the start: 36 parts

Commit message: commented all necessary in the Python code and renamed PCBs folder to PCBs_schematics
Parts:
- removed C?: C, symbol C
- added SW?: SW_SPDT, symbol SW_SPDT
- R?: value 100R -> 1k
Connections:
- net at R?.1, R?.1, U?.1 (IN+): now also SW?.1 (A); no longer BT?.1 (+)
- new net: BT?.1 (+), SW?.2 (B)
Other:
- moved on the sheet: BT?
Changed lines of the file:
@@
 P 3500 4350
 F 0 "R?" V 3580 4350 50  0000 C CNN
-F 1 "100R" V 3500 4350 50  0000 C CNN
+F 1 "1k" V 3500 4350 50  0000 C CNN
 F 2 "" V 3430 4350 50  0001 C CNN
 F 3 "" H 3500 4350 50  0001 C CNN
@@
 $EndComp
 $Comp
-L C C?
-U 1 1 5A3CDF1D
-P 9200 2500
-F 0 "C?" H 9225 2600 50  0000 L CNN
-F 1 "C" H 9225 2400 50  0000 L CNN
-F 2 "" H 9238 2350 50  0001 C CNN
-F 3 "" H 9200 2500 50  0001 C CNN
-	1    9200 2500
-	1    0    0    -1
-$EndComp
-$Comp
-L GND #PWR?
-U 1 1 5A3CE00A
-P 9200 2750
-F 0 "#PWR?" H 9200 2500 50  0001 C CNN
-F 1 "GND" H 9200 2600 50  0000 C CNN
-F 2 "" H 9200 2750 50  0001 C CNN
-F 3 "" H 9200 2750 50  0001 C CNN
-	1    9200 2750
-	1    0    0    -1
-$EndComp
-$Comp
 L +3.3V #PWR?
 U 1 1 5A3AD6C0
@@
 L Battery BT?
 U 1 1 5A3CFE67
-P 10450 3500
-F 0 "BT?" H 10550 3600 50  0000 L CNN
-F 1 "Battery" H 10550 3500 50  0000 L CNN
-F 2 "" V 10450 3560 50  0001 C CNN
-F 3 "" V 10450 3560 50  0001 C CNN
-	1    10450 3500
+P 10900 3500
+F 0 "BT?" H 11000 3600 50  0000 L CNN
+F 1 "Battery" H 11000 3500 50  0000 L CNN
+F 2 "" V 10900 3560 50  0001 C CNN
+F 3 "" V 10900 3560 50  0001 C CNN
+	1    10900 3500
 	1    0    0    -1
 $EndComp
@@
 	1850 1550 2250 1550
 Wire Wire Line
-	9850 3700 10450 3700
+	9850 3700 10900 3700
 Wire Wire Line
 	8300 750  8700 750
@@
 	9950 2150 9950 2100
 Wire Wire Line
-	9450 2300 9450 2350
-Wire Wire Line
-	9200 2350 9550 2350
-Wire Wire Line
 	6150 1700 6500 1700
 Wire Wire Line
@@
 	7500 5100 7500 5000
 Wire Wire Line
-	9200 2750 9200 2650
-Wire Wire Line
 	2450 4800 2450 5900
 Wire Wire Line
@@
 	10450 3300 10150 3300
 Connection ~ 10150 3300
-Connection ~ 9450 2350
 Wire Wire Line
 	10350 2500 10400 2500
@@
 Wire Wire Line
 	4600 4150 3500 4150
+Wire Wire Line
+	9550 2350 9450 2350
+Wire Wire Line
+	9450 2350 9450 2300
+$Comp
+L SW_SPDT SW?
+U 1 1 5A74538D
+P 10650 3200
+F 0 "SW?" H 10650 3370 50  0000 C CNN
+F 1 "SW_SPDT" H 10650 3000 50  0000 C CNN
+F 2 "" H 10650 3200 50  0001 C CNN
+F 3 "" H 10650 3200 50  0001 C CNN
+	1    10650 3200
+	-1   0    0    1
+$EndComp
+Wire Wire Line
+	10900 3300 10900 3200
+Wire Wire Line
+	10900 3200 10850 3200
 $EndSCHEMATC
