File: PCBs_schematics/Rover-general.sch (KiCad schematic (older format))
At the start: 36 parts

Commit message: added 6V buck-converter version to the schematic
Parts:
- removed U?: LM2576HVT-5, TO_SOT_Packages_THT:TO-220-5_Vertical, symbol LM2576HVT-5
- added C?: 100uF, symbol CP
- added C?: 33uF, symbol CP
- added C? (x2): 47uF, symbol CP
- added D?: D_Schottky, symbol D_Schottky
- added L?: 470uH, symbol INDUCTOR
- added R?: 10k, symbol R_Variable
- added R?: 2k, symbol R
- added U?: LM2576T-5, TO_SOT_Packages_THT:TO-220-5_Vertical, symbol LM2576T-5
- added U?: LM2576T-ADJ, TO_SOT_Packages_THT:TO-220-5_Vertical, symbol LM2576T-ADJ
Connections:
- net +12V: now also C?.1, U?.1 (VIN), U?.1 (VIN)
- net +5V: now also C?.2, C?.1, C?.1, U?.4 (FB); no longer C?.1
- net GND: now also C?.1, C?.2, C?.2, C?.2, C?.2, D?.2 (A), R?.1, U?.3 (GND), U?.3 (GND), U?.5 (~ON~/OFF), U?.5 (~ON~/OFF); no longer C?.2
- net at D?.1 (K), L?.1: now also U?.2 (OUT)
- new net: D?.1 (K), L?.1, U?.2 (OUT)
- new net: C?.1, L?.2, R?.2
- new net: R?.1, R?.2, U?.4 (FB)
Other:
- moved on the sheet: BT?, C?, R?, SW?, U?
