File: PCBs_schematics/General scheme/Rover.sch (KiCad schematic (older format))
At the start: 45 parts

Commit message: progress on the PCB
Parts:
- R?: value R_Variable -> 7756R
Changed lines of the file:
@@
 P 10850 2350
 F 0 "R?" V 10950 2250 50  0000 C CNN
-F 1 "R_Variable" V 10750 2300 50  0000 L CNN
+F 1 "7756R" V 10750 2300 50  0000 L CNN
 F 2 "" V 10780 2350 50  0001 C CNN
 F 3 "" H 10850 2350 50  0001 C CNN
