File: PCBs_schematics/PCB-Layout/Rover.kicad_pcb (KiCad board)
At the start: 2 copper layers, 93 x 135 mm, 49 parts, among them J1 ToF-sensor2, J2 Pi-15,17, J3 Conn_01x02, J4 Conn_01x04, J5 Conn_01x04, J6 Conn_01x03, J7 USB-conn, M1 Sensor-DC-motor, M2 Wheel-dc-motor, M3 Motor_Servo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

Commit message: edited pcb files for production
Parts:
- moved R5 0.75 mm to (44.5, 82.8)
