File: PCBs_schematics/PCB-Layout/out/pokus.kicad_pcb (KiCad board)
At the start: 2 copper layers, 93 x 135 mm, 49 parts, among them J1 ToF-sensor2, J2 Pi-15,17, J3 Conn_01x02, J4 Conn_01x04, J5 Conn_01x04, J6 Conn_01x03, J7 USB-conn, M1 Sensor-DC-motor, M2 Wheel-dc-motor, M3 Motor_Servo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

Commit message: more progress on the PCBs
Changed lines of the file:
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@@
   )
   (setup
-    (last_trace_width 1.5)
+    (last_trace_width 0.25)
     (user_trace_width 0.65)
     (user_trace_width 1)
@@
     (mod_text_size 1 1)
     (mod_text_width 0.15)
-    (pad_size 1.99898 1.99898)
-    (pad_drill 1.00076)
+    (pad_size 5.00126 5.00126)
+    (pad_drill 1)
     (pad_to_mask_clearance 0)
     (aux_axis_origin 0 0)
@@
     (fp_line (start -2.6162 -4.1148) (end -2.1336 -5.1816) (layer Cmts.User) (width 0.381))
     (fp_line (start -2.1336 -5.1816) (end -2.1336 -3.6322) (layer Cmts.User) (width 0.381))
-    (pad 1 thru_hole circle (at 0 0 270) (size 5.00126 5.00126) (drill 2.49936) (layers *.Cu *.Mask)
+    (pad 1 thru_hole circle (at 0 0 270) (size 5.00126 5.00126) (drill 1) (layers *.Cu *.Mask)
       (net 7 "Net-(C3-Pad1)") (thermal_width 1.5))
-    (pad 2 thru_hole circle (at 10.16 0 270) (size 5.00126 5.00126) (drill 2.49936) (layers *.Cu *.Mask)
+    (pad 2 thru_hole circle (at 10.16 0 270) (size 5.00126 5.00126) (drill 1) (layers *.Cu *.Mask)
       (net 3 "Net-(C1-Pad1)") (thermal_width 1.5))
   )
@@
     (fp_line (start -2.6162 -4.1148) (end -2.1336 -5.1816) (layer Cmts.User) (width 0.381))
     (fp_line (start -2.1336 -5.1816) (end -2.1336 -3.6322) (layer Cmts.User) (width 0.381))
-    (pad 1 thru_hole circle (at 0 0 270) (size 5.00126 5.00126) (drill 2.49936) (layers *.Cu *.Mask)
+    (pad 1 thru_hole circle (at 0 0 270) (size 5.00126 5.00126) (drill 1) (layers *.Cu *.Mask)
       (net 8 "Net-(C3-Pad2)") (thermal_width 1.5))
-    (pad 2 thru_hole circle (at 10.16 0 270) (size 5.00126 5.00126) (drill 2.49936) (layers *.Cu *.Mask)
+    (pad 2 thru_hole circle (at 10.16 0 270) (size 5.00126 5.00126) (drill 1) (layers *.Cu *.Mask)
       (net 4 "Net-(C1-Pad2)") (thermal_width 1.5))
   )
@@
     (fp_line (start -2.6162 -4.1148) (end -2.1336 -5.1816) (layer Cmts.User) (width 0.381))
     (fp_line (start -2.1336 -5.1816) (end -2.1336 -3.6322) (layer Cmts.User) (width 0.381))
-    (pad 1 thru_hole circle (at 0 0 270) (size 5.00126 5.00126) (drill 2.49936) (layers *.Cu *.Mask)
+    (pad 1 thru_hole circle (at 0 0 270) (size 5.00126 5.00126) (drill 1) (layers *.Cu *.Mask)
       (net 9 "Net-(C4-Pad1)") (thermal_width 1.5))
-    (pad 2 thru_hole circle (at 10.16 0 270) (size 5.00126 5.00126) (drill 2.49936) (layers *.Cu *.Mask)
+    (pad 2 thru_hole circle (at 10.16 0 270) (size 5.00126 5.00126) (drill 1) (layers *.Cu *.Mask)
       (net 5 "Net-(C2-Pad1)") (thermal_width 1.5))
   )
@@
     (fp_line (start -2.6162 -4.1148) (end -2.1336 -5.1816) (layer Cmts.User) (width 0.381))
     (fp_line (start -2.1336 -5.1816) (end -2.1336 -3.6322) (layer Cmts.User) (width 0.381))
-    (pad 1 thru_hole circle (at 0 0 270) (size 5.00126 5.00126) (drill 2.49936) (layers *.Cu *.Mask)
+    (pad 1 thru_hole circle (at 0 0 270) (size 5.00126 5.00126) (drill 1) (layers *.Cu *.Mask)
       (net 10 "Net-(C4-Pad2)") (thermal_width 1.5))
-    (pad 2 thru_hole circle (at 10.16 0 270) (size 5.00126 5.00126) (drill 2.49936) (layers *.Cu *.Mask)
+    (pad 2 thru_hole circle (at 10.16 0 270) (size 5.00126 5.00126) (drill 1) (layers *.Cu *.Mask)
       (net 6 "Net-(C2-Pad2)") (thermal_width 1.5))
   )
