File: PCBs_schematics/General-scheme/Rover.sch (KiCad schematic (older format))
At the start: 45 parts

Commit message: renamed folder and added value to the crytal
Parts:
- Y?: value Crystal -> 16.000MHz
Changed lines of the file:
@@
 P 3300 6950
 F 0 "Y?" H 3300 7100 50  0000 C CNN
-F 1 "Crystal" H 3300 6800 50  0000 C CNN
+F 1 "16.000MHz" H 3300 6800 50  0000 C CNN
 F 2 "" H 3300 6950 50  0001 C CNN
 F 3 "" H 3300 6950 50  0001 C CNN
